File: hardware/controller/controller.kicad_sch (KiCad schematic)
At the start: 77 parts, among them J1 USB_C_Receptacle_USB2.0_16P, J2 Micro_SD_Card_Det_Hirose_DM3AT, J3 Display, SW1 Reset, SW2 Boot, SW3 SW_SPDT, SW4 EStop, U2 SX1262IMLTRT, U3 MP2672AGD-0000-Z, U4 PE4259, U5 LMR51625XDDCR, U6 ESP32-S3-MINI-1, Y2 32MHz

Commit message: routing board
Parts:
- added Q1: AO3400A, Package_TO_SOT_SMD:SOT-23, symbol Transistor_FET:AO3400A
- added R27: 10K, Resistor_SMD:R_0402_1005Metric, symbol Device:R
Connections:
- net GND: now also R1.D, R2.D, Q1.2 (S); no longer R1.B, R2.B, U5.4 (GND)
- net JOY_1_BTN: now also R1.A; no longer R1.C
- net JOY_2_BTN: now also R2.A; no longer R2.C
- net MISO: now also U6.17 (IO13)
- net MOSI: now also U6.15 (IO11)
- net SCK: now also U6.16 (IO12)
- net SX_CS: now also U6.14 (IO10)
- net VCC: now also C15.1, U5.2 (EN), U5.3 (VIN), R27.1; no longer SW3.2 (B)
- new net: R27.2, SW3.2 (B)
- new net: Q1.1 (G), SW3.3 (C)
- new net: Q1.3 (D), U5.4 (GND)
- no-connect marks 22 -> 20
Other:
- moved on the sheet: C15, C16, C24, C25, L5, R23, R24, SW3, U5

Commit message: finished first version
Parts:
- removed BT2: Battery_Cell, Battery:BatteryHolder_MPD_BH-18650-PC, symbol Device:Battery_Cell
- removed C23: 22uF, Capacitor_SMD:C_0805_2012Metric, symbol Device:C
- removed C24, C25: 33uF, Capacitor_SMD:C_0603_1608Metric, symbol Device:C
- removed D2: LED, LED_THT:LED_D3.0mm, symbol Device:LED
- removed L5: 10uH, Inductor_SMD:L_APV_ANR4010, symbol Device:L
- removed R1, R2: THB001P, Imports:THB001P_CNK, symbol Imports:THB001P
- removed R20: 2K, Resistor_SMD:R_0402_1005Metric, symbol Device:R
- removed R23: 31.6K, Resistor_SMD:R_0402_1005Metric, symbol Device:R
- removed R24: 10.2, Resistor_SMD:R_0402_1005Metric, symbol Device:R
- removed U3: MP2672AGD-0000-Z, Imports:QFN-18_MP2672A_MNP, symbol Imports:MP2672AGD-0000-Z
- removed U4: PE4259, Package_TO_SOT_SMD:SOT-363_SC-70-6, symbol Imports:PE4259
- removed U5: LMR51625XDDCR, Package_TO_SOT_SMD:SOT-23-6, symbol Imports:LMR51625XDDCR
- added R1, R2: THB001P, controller:THB001P_CNK, symbol controller:THB001P
- added U1: BQ25895RTW, Package_DFN_QFN:Texas_RTW_WQFN-24-1EP_4x4mm_P0.5mm_EP2.7x2.7mm_ThermalVias, symbol Battery_Management:BQ25895RTW
- added U3: AMS1117-3.3, Package_TO_SOT_SMD:SOT-223-3_TabPin2, symbol Regulator_Linear:AMS1117-3.3
- added U4: PE4259, Package_TO_SOT_SMD:SOT-363_SC-70-6, symbol controller:PE4259
- BT1: value Battery_Cell -> Battery
- C15: value 2.2uF -> 1uF
- C16: value 0.1uF -> 47nF
- C17: value 0.1uF -> 22uF; footprint Capacitor_SMD:C_0402_1005Metric -> Capacitor_SMD:C_0603_1608Metric
- C18: value 10uF -> 22uF
- C19: value 22uF -> 4.7uF; footprint Capacitor_SMD:C_0603_1608Metric -> Capacitor_SMD:C_0402_1005Metric
- C20: value 22uF -> 10uF
- C21, C22: value 1uF -> 10uF; footprint Capacitor_SMD:C_0402_1005Metric -> Capacitor_SMD:C_0603_1608Metric
- D1: footprint LED_THT:LED_D3.0mm -> LED_SMD:LED_0603_1608Metric
- L4: value 1.5uH -> 2.2uH
- R13: value 10K -> 5.2K
- R14: value 28.7K -> 30.1K
- R15: value 2K -> 5.1K
- R16: value 2K -> 10K
- R17: value 12K -> 10K
- R18: value 12.62K -> 10K
- R19: value 3K -> 260
- SW4: footprint Button_Switch_SMD:SW_Push_SPST_NO_Alps_SKRK -> Connector_Wire:SolderWire-0.1sqmm_1x02_P3.6mm_D0.4mm_OD1mm
- TH1: value NTCG -> Thermistor; footprint Resistor_SMD:R_0402_1005Metric -> Resistor_SMD:R_0201_0603Metric
Connections:
- net +3.3V: now also C17.1, R16.1, R17.1, R18.1, R1.1, R1.1', R2.1, R2.1', U3.2 (VO), U4.6 (VDD); no longer R15.1, R16.2
- net GND: now also BT1.2 (-), C17.2, R19.2, R1.3, R1.3', R1.D, R2.3, R2.3', R2.D, U1.17 (PGND), U1.18 (PGND), U1.25 (PGND), U4.2 (GND); no longer R17.2
- net JOY_1_BTN: now also R2.A
- net JOY_1_X: now also R2.2'
- net JOY_1_Y: now also R2.2
- net JOY_2_BTN: now also R1.A
- net JOY_2_X: now also R1.2'
- net JOY_2_Y: now also R1.2
- net SCL: now also R17.2, U1.6 (SDA)
- net SDA: now also R16.2, U1.5 (SCL)
- net SD_DAT0: no longer U6.35 (IO39)
- net SD_DAT1: no longer U6.36 (IO40)
- net SD_DET_1: now also U6.35 (IO39); no longer J2.10 (DET_A)
- net SX_BUSY: now also U6.18 (IO14)
- net SX_DIO1: now also U6.19 (IO15)
- net SX_RST: now also U6.20 (IO16)
- net VBUS: now also C15.1, U1.1 (VBUS); no longer C18.1, L4.1, R13.1
- net VCC: now also C18.1, C22.1, D1.2 (A), L4.2, U1.15 (SYS), U1.16 (SYS), U3.3 (VI); no longer C15.1, C19.1, C20.1
- net BQ_INT: now reaches U6.37 (IO41)
- net BQ_INT: now also R18.2, U1.7 (~{INT})
- net BQ_CE: now reaches U6.38 (IO42)
- net BQ_CE: now also U1.9 (~{CE})
- net at R13.2, R14.1: now also TH1.1, U1.11 (TS)
- net at FL1.8 (SW_RFO): now also U4.1 (RF1)
- net at FL1.6 (SW_RFI): now also U4.3 (RF2)
- net at C9.1, R4.2: now also U4.4 (CTRL)
- net at C10.1: now also U4.5 (RFIN)
- net at D1.1 (K): now also R15.2
- net at BT1.1 (+), R21.1: now also C20.1, U1.13 (BAT), U1.14 (BAT)
- net at R19.1: now also U1.10 (ILIM); no longer R18.2
- net at Q1.3 (D): now also U3.1 (GND)
- net at C16.2: now also U1.21 (BTST)
- net at C16.1: now also L4.1, U1.19 (SW), U1.20 (SW)
- new net: C19.1, R13.1, U1.22 (REGN)
- new net: R15.1, U1.4 (STAT)
- new net SD_DET_0: J2.10 (DET_A), U6.36 (IO40)
- no-connect marks 20 -> 22
Other:
- note added: "Regulator"
- note removed: "Buck Regulator"
- note removed: "Configured for: 1A charge 4.675V min input volage"
- note removed: "Couldn't figure out the exact calculation for the thermistor voltage divider but this should be acceptable"
- moved on the sheet: Q1, R21, R22, R27, SW3

Commit message: finished board
Changed lines of the file:
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@@
 	(text "Regulator"
 		(exclude_from_sim no)
-		(at 294.132 15.748 0)
+		(at 288.036 14.986 0)
 		(effects
 			(font

Commit message: added tranceiver and joystick
Parts:
- removed AE1: Antenna, Connector_Coaxial:SMA_Amphenol_901-143_Horizontal, symbol Device:Antenna
- added C23: 0.1uF, Capacitor_SMD:C_0402_1005Metric, symbol Device:C
- added J4: Conn_Coaxial, Connector_Coaxial:SMA_Amphenol_901-143_Horizontal, symbol Connector:Conn_Coaxial
- added SW5: BTN_2, Connector_Wire:SolderWire-0.1sqmm_1x02_P3.6mm_D0.4mm_OD1mm, symbol Switch:SW_Push
- SW4: value EStop -> BTN_1
Connections:
- net GND: now also C23.1, J4.2 (Ext), SW5.1
- net SX_BUSY: now also U6.19 (IO15); no longer U6.18 (IO14)
- net SX_DIO1: now also U6.20 (IO16); no longer U6.19 (IO15)
- net SX_RST: now also U6.18 (IO14); no longer U6.20 (IO16)
- net BTN_1: now reaches U6.21 (IO17)
- net BTN_1: now also C26.2, SW4.2
- net at C12.1, L3.2: now also J4.1 (In)
- removed net ESTOP: C26.2, SW4.2, U6.22 (IO18)
- new net BTN_2: C23.2, SW5.2, U6.22 (IO18)
- no-connect marks 22 -> 21
Other:
- note added: "Buttons"
- note removed: "EStop Button"
- moved on the sheet: C26, SW4

Commit message: updated controller pcb
Parts:
- removed C1, C2: 0.1uF, Capacitor_SMD:C_0402_1005Metric, symbol Device:C
- removed C10: 39pF, Capacitor_SMD:C_0402_1005Metric, symbol Device:C
- removed C11, C12: 3.3pF, Capacitor_SMD:C_0402_1005Metric, symbol Device:C
- removed C3: 470nF, Capacitor_SMD:C_0402_1005Metric, symbol Device:C
- removed C7: 47nF, Capacitor_SMD:C_0402_1005Metric, symbol Device:C
- removed C8: 47pF, Capacitor_SMD:C_0402_1005Metric, symbol Device:C
- removed C9: 1nF, Capacitor_SMD:C_0402_1005Metric, symbol Device:C
- removed FL1: 0900FM15K0039, RF_Converter:Balun_Johanson_0900FM15K0039, symbol Filter:0900FM15K0039
- removed J4: Conn_Coaxial, Connector_Coaxial:SMA_Amphenol_901-143_Horizontal, symbol Connector:Conn_Coaxial
- removed L1: 15uH, Inductor_SMD:L_0402_1005Metric, symbol Device:L
- removed L2: 47nH, Inductor_SMD:L_0402_1005Metric, symbol Device:L
- removed L3: 9.1nH, Inductor_SMD:L_0402_1005Metric, symbol Device:L
- removed R4: 100, Resistor_SMD:R_0402_1005Metric, symbol Device:R
- removed U2: SX1262IMLTRT, Package_DFN_QFN:QFN-24-1EP_4x4mm_P0.5mm_EP2.6x2.6mm, symbol RF:SX1262IMLTRT
- removed U4: PE4259, Package_TO_SOT_SMD:SOT-363_SC-70-6, symbol controller:PE4259
- removed Y2: 32MHz, Crystal:Crystal_SMD_3225-4Pin_3.2x2.5mm, symbol Device:Crystal_GND24
- added J4: Tranceiver Data, Connector_JST:JST_XH_B4B-XH-A_1x04_P2.50mm_Vertical, symbol Connector_Generic:Conn_01x04
- added J5: Tranceiver Boot/Rst, Connector_JST:JST_XH_B2B-XH-A_1x02_P2.50mm_Vertical, symbol Connector_Generic:Conn_01x02
- D1: footprint LED_SMD:LED_0603_1608Metric -> LED_THT:LED_D5.0mm
Connections:
- net +3.3V: now also J4.1 (Pin_1)
- net GND: now also J4.2 (Pin_2)
- net ESP_TX: now reaches U6.39 (TXD0)
- net ESP_TX: now also J4.4 (Pin_4)
- net ESP_RX: now reaches U6.40 (RXD0)
- net ESP_RX: now also J4.3 (Pin_3)
- net MISO: no longer names the net of U6.17 (IO13)
- net MOSI renamed STM32_BOOT
- net STM32_BOOT: now also J5.2 (Pin_2)
- net SCK: no longer names the net of U6.16 (IO12)
- net SX_BUSY: no longer names the net of U6.19 (IO15)
- net SX_CS renamed STM32_RST
- net STM32_RST: now also J5.1 (Pin_1)
- net SX_DIO1: no longer names the net of U6.20 (IO16)
- net SX_RST: no longer names the net of U6.18 (IO14)
- no-connect marks 21 -> 24
Other:
- note added: "Tranceiver Module"
- note removed: "SX1262 LoRa Module"
- moved on the sheet: BT1, C13, C14, C15, C16, C17, C18, C19, C20, C21, C22, C23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

Commit message: cleaning up controller pcb
Parts:
- J3: footprint Connector_JST:JST_PH_S4B-PH-K_1x04_P2.00mm_Horizontal -> Connector_JST:JST_XH_B4B-XH-A_1x04_P2.50mm_Vertical
Changed lines of the file:
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@@
 			)
 		)
-		(property "Footprint" "Connector_JST:JST_PH_S4B-PH-K_1x04_P2.00mm_Horizontal"
+		(property "Footprint" "Connector_JST:JST_XH_B4B-XH-A_1x04_P2.50mm_Vertical"
 			(at 269.24 36.83 0)
 			(effects
