File: hardware/controller/controller.kicad_sch (KiCad schematic)
At the start: 56 parts, among them J1 USB_C_Receptacle_USB2.0_16P, J2 Micro_SD_Card_Det_Hirose_DM3AT, J3 Display, J4 Tranceiver Data, J5 Tranceiver Boot/Rst, Q1 AO3400A, SW1 Reset, SW2 Boot, SW3 SW_SPDT, SW4 BTN_1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

Commit message: changed switch circuit
Connections:
- net GND: now also U3.1 (GND); no longer Q1.2 (S)
- net VCC: now also Q1.3 (D); no longer C18.1, U3.3 (VI)
- new net: C18.1, Q1.2 (S), U3.3 (VI)
Other:
- moved on the sheet: C13, C14, C17, C18, C23, C26, Q1, R27, SW1, SW2, SW3, SW4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

Commit message: fixed switch and joysticks
Parts:
- removed Q1: AO3400A, Package_TO_SOT_SMD:SOT-23, symbol Transistor_FET:AO3400A
- added C1, C2: 0.1uF, Capacitor_SMD:C_0402_1005Metric, symbol Device:C
- added Q1: AO3401A, Package_TO_SOT_SMD:SOT-23, symbol Transistor_FET:AO3401A
- added R4: 100, Resistor_SMD:R_0402_1005Metric, symbol Device:R
- R27: value 10K -> 100
Connections:
- net +3.3V: now also C2.1
- net GND: now also C1.2, C2.2, R4.2
- net VCC: now also Q1.2 (S)
- net at C18.1, U3.3 (VI): now also C1.1, Q1.3 (D)
- net at SW3.1 (A): now also R27.2
- net at SW3.2 (B): now also Q1.1 (G); no longer R27.2
- net at SW3.3 (C): now also R4.1
- no-connect marks 24 -> 23
Other:
- moved on the sheet: C17, C18, R27, SW3, U3

Commit message: fixed usb
Parts:
- R25, R26: value 27K -> 27
Changed lines of the file:
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@@
 			)
 		)
-		(property "Value" "27K"
+		(property "Value" "27"
 			(at 163.83 129.286 90)
 			(effects
@@
 			)
 		)
-		(property "Value" "27K"
+		(property "Value" "27"
 			(at 163.576 122.428 90)
 			(effects

Commit message: added production files
Parts:
- R19: value 260 -> 200
Changed lines of the file:
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@@
 			)
 		)
-		(property "Value" "260"
+		(property "Value" "200"
 			(at 97.79 68.58 0)
 			(effects
