File: hardware/controller/controller.kicad_pcb (KiCad board)
At the start: 4 copper layers, 77 parts, among them J1 USB_C_Receptacle_USB2.0_16P, J2 Micro_SD_Card_Det_Hirose_DM3AT, J3 Display, SW1 Reset, SW2 Boot, SW3 SW_SPDT, SW4 EStop, U2 SX1262IMLTRT, U3 MP2672AGD-0000-Z, U4 PE4259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

Commit message: routing board
Parts:
- added Q1: AO3400A, Package_TO_SOT_SMD:SOT-23, F.Cu at (133.9, 126.3)
- added R27: 10K, Resistor_SMD:R_0402_1005Metric, F.Cu at (140.2, 126.5)
- moved C13 108.3 mm to (246.9, 132.8)
- moved C26 108.3 mm to (246.8, 126.9)
- moved SW1 108.3 mm to (246.8, 142.2)
- moved SW2 108.3 mm to (246.8, 135.2)
- moved SW4 108.3 mm to (246.8, 129.2)
- moved C14 108.3 mm to (247.0, 139.9)
- moved R3 87.8 mm to (182.7, 141.9), turned to 90 degrees
- moved C6 85.6 mm to (181.2, 123.2), turned to 90 degrees
- moved C4 85.5 mm to (181.4, 142.0), turned to 90 degrees
- moved C5 82.9 mm to (179.9, 123.9), turned to 90 degrees
- moved J3 81.8 mm to (88.0, 116.0), turned to -90 degrees
- moved U6 77.2 mm to (178.2, 132.8), turned to -90 degrees
- moved R15 56.1 mm to (123.0, 153.5), turned to -90 degrees
- moved D1 55.9 mm to (120.5, 157.0)
- moved R25 54.2 mm to (166.7, 132.8), turned to 180 degrees
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Connections:
- C15 pad 1: Net-(SW3-C) -> VCC
- R1 pad A: unconnected-(R1-PadA) -> /JOY_1_BTN
- R1 pad B: GND -> unconnected-(R1-PadB)
- R1 pad C: /JOY_1_BTN -> unconnected-(R1-PadC)
- R1 pad D: unconnected-(R1-PadD) -> GND
- R2 pad A: unconnected-(R2-PadA) -> /JOY_2_BTN
- R2 pad B: GND -> unconnected-(R2-PadB)
- R2 pad C: /JOY_2_BTN -> unconnected-(R2-PadC)
- R2 pad D: unconnected-(R2-PadD) -> GND
- SW3 pad 2: VCC -> Net-(SW3-B)
- SW3 pad 3: Net-(SW3-C) -> Net-(Q1-G)
- U5 pad 2: Net-(SW3-C) -> VCC
- U5 pad 3: Net-(SW3-C) -> VCC
- U5 pad 4: GND -> Net-(Q1-D)
- U6 pad 14: unconnected-(U6-IO10-Pad14) -> /SX_CS
- U6 pad 15: unconnected-(U6-IO11-Pad15) -> /MOSI
- U6 pad 16: unconnected-(U6-IO12-Pad16) -> /SCK
- U6 pad 17: unconnected-(U6-IO13-Pad17) -> /MISO
Routing:
- net +3.3V: track 0.00 -> 68.1 mm
- net Net-(BT1--): track 0.00 -> 65.9 mm, vias 0 -> 1
- net Net-(BT1-+): track 0.00 -> 61.0 mm, vias 0 -> 1
- net Net-(R19-Pad2): track 0.00 -> 46.9 mm, vias 0 -> 1
- net /USB_D-: track 0.00 -> 43.5 mm
- net /USB_D+: track 0.00 -> 43.5 mm
- net /SD_DAT0: track 1.92 -> 28.3 mm
- net /SD_CLK: track 1.84 -> 24.7 mm
- net Net-(D1-K): track 0.00 -> 22.8 mm, vias 0 -> 1
- net Net-(D2-K): track 0.00 -> 22.2 mm, vias 0 -> 1
- net /SD_CMD: track 1.76 -> 21.3 mm
- net VBUS: track 0.00 -> 19.3 mm
- net Net-(U3-VLIM): track 0.00 -> 18.2 mm
- net /SD_DAT3: track 1.75 -> 19.5 mm
- net /SD_DAT2: track 1.75 -> 17.5 mm
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Other:
- board outline added: 125 x 95 mm

Commit message: finished first version
Parts:
- removed BT2: Battery_Cell, Battery:BatteryHolder_MPD_BH-18650-PC
- removed C23: 22uF, Capacitor_SMD:C_0805_2012Metric
- removed C24, C25: 33uF, Capacitor_SMD:C_0603_1608Metric
- removed D2: LED, LED_THT:LED_D3.0mm
- removed L5: 10uH, Inductor_SMD:L_APV_ANR4010
- removed R20: 2K, Resistor_SMD:R_0402_1005Metric
- removed R23: 31.6K, Resistor_SMD:R_0402_1005Metric
- removed R24: 10.2, Resistor_SMD:R_0402_1005Metric
- removed U5: LMR51625XDDCR, Package_TO_SOT_SMD:SOT-23-6
- added U1: BQ25895RTW, Package_DFN_QFN:Texas_RTW_WQFN-24-1EP_4x4mm_P0.5mm_EP2.7x2.7mm_ThermalVias, F.Cu at (131.1, 145.8)
- BT1: value Battery_Cell -> Battery
- C15: value 2.2uF -> 1uF
- C16: value 0.1uF -> 47nF
- C17: value 0.1uF -> 22uF; footprint Capacitor_SMD:C_0402_1005Metric -> Capacitor_SMD:C_0603_1608Metric
- C18: value 10uF -> 22uF
- C19: value 22uF -> 4.7uF; footprint Capacitor_SMD:C_0603_1608Metric -> Capacitor_SMD:C_0402_1005Metric
- C20: value 22uF -> 10uF
- C21, C22: value 1uF -> 10uF; footprint Capacitor_SMD:C_0402_1005Metric -> Capacitor_SMD:C_0603_1608Metric
- D1: footprint LED_THT:LED_D3.0mm -> LED_THT:LED_D5.0mm
- J3: footprint Connector_JST:JST_PH_S4B-PH-K_1x04_P2.00mm_Horizontal -> Connector_JST:JST_PH_B4B-PH-K_1x04_P2.00mm_Vertical
- L4: value 1.5uH -> 2.2uH; footprint Inductor_SMD:L_6.3x6.3_H3 -> Inductor_SMD:L_7.3x7.3_H3.5
- R1, R2: footprint Imports:THB001P_CNK -> controller:THB001P_CNK
- R13: value 10K -> 5.2K
- R14: value 28.7K -> 30.1K
- R15: value 2K -> 5.1K
- R16: value 2K -> 10K
- R17: value 12K -> 10K
- R18: value 12.62K -> 10K
- R19: value 3K -> 260
- SW4: footprint Button_Switch_SMD:SW_Push_SPST_NO_Alps_SKRK -> Connector_Wire:SolderWire-0.1sqmm_1x02_P3.6mm_D0.4mm_OD1mm
- TH1: value NTCG -> Thermistor; footprint Resistor_SMD:R_0402_1005Metric -> Resistor_SMD:R_0201_0603Metric
- U3: value MP2672AGD-0000-Z -> AMS1117-3.3; footprint Imports:QFN-18_MP2672A_MNP -> Package_TO_SOT_SMD:SOT-223-3_TabPin2
- moved SW2 129.4 mm to (118.2, 149.5)
- moved C13 129.4 mm to (118.2, 147.1)
- moved SW4 86.7 mm to (160.1, 130.5)
- moved C26 84.8 mm to (162.0, 128.5)
- moved C14 79.6 mm to (168.3, 151.9)
- moved SW1 79.0 mm to (168.2, 149.6)
- moved R16 53.3 mm to (172.3, 123.9), turned to -90 degrees
- moved R17 39.9 mm to (171.3, 123.9), turned to -90 degrees
- moved C16 19.7 mm to (127.7, 145.0), turned to -90 degrees
- moved C15 19.7 mm to (129.2, 149.0), turned to 180 degrees
- moved C18 15.9 mm to (125.8, 133.8)
- moved C19 14.2 mm to (127.3, 146.5), turned to 180 degrees
- moved TH1 13.8 mm to (143.2, 111.0)
- moved C17 12.0 mm to (124.4, 130.0), turned to -90 degrees
- moved BT1 9.80 mm to (179.7, 99.2)
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Connections:
- BT1 pad 2: Net-(BT1--) -> GND
- C15 pad 1: VCC -> VBUS
- C16 pad 1: Net-(U5-CB) -> Net-(C16-Pad1)
- C17 pad 1: Net-(C17-Pad1) -> +3.3V
- C17 pad 2: Net-(U3-BST) -> GND
- C18 pad 1: VBUS -> VCC
- C19 pad 1: VCC -> Net-(U1-REGN)
- C20 pad 1: VCC -> Net-(BT1-+)
- C22 pad 1: Net-(U3-VCC) -> VCC
- D1 pad 2: Net-(D1-A) -> VCC
- J2 pad 10: /SD_DET_1 -> /SD_DET_0
- L4 pad 1: VBUS -> Net-(C16-Pad1)
- L4 pad 2: Net-(C17-Pad1) -> VCC
- R1 pad 2: /JOY_1_X -> /JOY_2_Y
- R1 pad 2': /JOY_1_Y -> /JOY_2_X
- R1 pad A: /JOY_1_BTN -> /JOY_2_BTN
- R13 pad 1: VBUS -> Net-(U1-REGN)
- R13 pad 2: Net-(U3-VLIM) -> Net-(U1-TS)
- R14 pad 1: Net-(U3-VLIM) -> Net-(U1-TS)
- R15 pad 1: +3.3V -> Net-(U1-STAT)
- R15 pad 2: Net-(D1-A) -> Net-(D1-K)
- R16 pad 1: Net-(D2-A) -> +3.3V
- R16 pad 2: +3.3V -> /SDA
- R17 pad 1: Net-(U3-ISET) -> +3.3V
- R17 pad 2: GND -> /SCL
- R18 pad 1: Net-(U3-VCC) -> +3.3V
- R18 pad 2: Net-(U3-NTC) -> /BQ_INT
- R19 pad 1: Net-(U3-NTC) -> Net-(U1-ILIM)
- R19 pad 2: Net-(R19-Pad2) -> GND
- R2 pad 2: /JOY_2_X -> /JOY_1_Y
- R2 pad 2': /JOY_2_Y -> /JOY_1_X
- R2 pad A: /JOY_2_BTN -> /JOY_1_BTN
- TH1 pad 1: Net-(R19-Pad2) -> Net-(U1-TS)
- U3 pad 1: VBUS -> Net-(Q1-D)
- U3 pad 2: Net-(C17-Pad1) -> +3.3V
- U3 pad 3: Net-(U3-BST) -> VCC
- U6 pad 18: unconnected-(U6-IO14-Pad18) -> /SX_BUSY
- U6 pad 19: unconnected-(U6-IO15-Pad19) -> /SX_DIO1
- U6 pad 20: unconnected-(U6-IO16-Pad20) -> /SX_RST
- U6 pad 35: /SD_DAT0 -> /SD_DET_1
- U6 pad 36: /SD_DAT1 -> /SD_DET_0
- U6 pad 37: unconnected-(U6-IO41-Pad37) -> /BQ_INT
- U6 pad 38: unconnected-(U6-IO42-Pad38) -> /BQ_CE
Routing:
- net /SDA: track 0.00 -> 114.0 mm, vias 0 -> 2
- net /SCL: track 0.00 -> 113.7 mm, vias 0 -> 2
- net /JOY_2_Y: track 0.00 -> 105.4 mm, vias 0 -> 1
- net /JOY_2_BTN: track 0.00 -> 101.6 mm, vias 0 -> 1
- net /JOY_2_X: track 0.00 -> 90.7 mm, vias 0 -> 1
- net /BOOT: track 0.00 -> 72.7 mm, vias 0 -> 2
- net GND: track 0.78 -> 69.3 mm, vias 0 -> 248
- net Net-(BT1--): track 65.9 -> 0.00 mm, vias 1 -> 0
- net /SX_RST: track 0.00 -> 52.0 mm, vias 0 -> 2
- net /SX_CS: track 0.00 -> 50.6 mm
- net /BQ_INT: track 0.00 -> 50.4 mm, vias 0 -> 2
- net /SCK: track 0.00 -> 49.6 mm, vias 0 -> 2
- net /SX_BUSY: track 0.00 -> 49.3 mm
- net /MISO: track 0.00 -> 49.2 mm
- net /SX_DIO1: track 0.00 -> 49.2 mm
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- added copper zone on In2.Cu, net +3.3V
- added copper zone on B.Cu, net GND
- added copper zone on F.Cu, net GND
- added copper zone on In1.Cu, net GND

Commit message: finished board
Parts:
- added REF**: MountingHole_3.2mm_M3, MountingHole:MountingHole_3.2mm_M3, F.Cu at (110.7, 74.5)
- added REF**: MountingHole_3.2mm_M3, MountingHole:MountingHole_3.2mm_M3, F.Cu at (110.7, 149.6)
- added REF**: MountingHole_3.2mm_M3, MountingHole:MountingHole_3.2mm_M3, F.Cu at (175.7, 149.6)
- added REF**: MountingHole_3.2mm_M3, MountingHole:MountingHole_3.2mm_M3, F.Cu at (175.7, 74.5)
Connections:
- AE1 pad 2: (no net) -> GND
Routing:
- net /EN: track 21.4 -> 22.0 mm
- net GND: vias 248 -> 251

Commit message: started cad
Parts:
- moved R1 2.03 mm to (94.1, 88.6)
- moved C13 0.05 mm to (118.2, 147.2)
- moved C14 0.05 mm to (168.3, 151.8)
- moved SW2 0.05 mm to (118.2, 149.6)
Routing:
- net +3.3V: track 60.1 -> 32.5 mm
- net /JOY_2_Y: track 105.4 -> 102.9 mm
- net /JOY_2_X: track 90.7 -> 89.3 mm
- net /JOY_2_BTN: track 101.6 -> 100.3 mm
- net GND: vias 251 -> 252
Changed lines of the file:
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@@
 	(footprint "controller:THB001P_CNK"
 		(layer "F.Cu")
-		(at 92.050599 88.604)
+		(at 94.081599 88.604)
 		(tags "THB001P ")
 		(property "Reference" "R1"
@@
 	(footprint "Button_Switch_SMD:SW_Push_SPST_NO_Alps_SKRK"
 		(layer "F.Cu")
-		(at 118.2 149.5)
+		(at 118.2 149.55)
 		(descr "http://www.alps.com/prod/info/E/HTML/Tact/SurfaceMount/SKRK/SKRKAHE020.html")
 		(tags "SMD SMT button")
@@
 		(model "${KICAD9_3DMODEL_DIR}/LED_THT.3dshapes/LED_D5.0mm.step"
 			(offset
-				(xyz 0 0 0)
+				(xyz 0 0 -3)
 			)
 			(scale
@@
 			)
 			(rotate
-				(xyz 0 0 0)
+				(xyz -0 -0 -0)
 			)
 		)
@@
 	(footprint "Capacitor_SMD:C_0402_1005Metric"
 		(layer "F.Cu")
-		(at 118.245 147.125)
+		(at 118.245 147.175)
 		(descr "Capacitor SMD 0402 (1005 Metric), square (rectangular) end terminal, IPC-7351 nominal, (Body size source: IPC-SM-782 page 76, https://www.pcb-3d.com/wordpress/wp-content/uploads/ipc-sm-782a_amendment_1_and_2.pdf), generated with kicad-footprint-generator")
 		(tags "capacitor")
@@
 	(footprint "Button_Switch_SMD:SW_Push_SPST_NO_Alps_SKRK"
 		(layer "F.Cu")
-		(at 168.2 149.6)
+		(at 168.2 149.55)
 		(descr "http://www.alps.com/prod/info/E/HTML/Tact/SurfaceMount/SKRK/SKRKAHE020.html")
 		(tags "SMD SMT button")
@@
 	(footprint "Capacitor_SMD:C_0402_1005Metric"
 		(layer "F.Cu")
-		(at 168.32 151.9)
+		(at 168.32 151.85)
 		(descr "Capacitor SMD 0402 (1005 Metric), square (rectangular) end terminal, IPC-7351 nominal, (Body size source: IPC-SM-782 page 76, https://www.pcb-3d.com/wordpress/wp-content/uploads/ipc-sm-782a_amendment_1_and_2.pdf), generated with kicad-footprint-generator")
 		(tags "capacitor")
@@
 	)
 	(via
+		(at 89 98)
+		(size 0.6)
+		(drill 0.3)
+		(layers "F.Cu" "B.Cu")
+		(free yes)
+		(net 4)
+	)
+	(via
 		(at 144.25 75.25)
 		(size 0.6)
@@
 	)
 	(segment
-		(start 197.415599 93.604)
-		(end 203.645599 99.834)
-		(width 0.4)
-		(layer "B.Cu")
-		(net 5)
-	)
-	(segment
-		(start 197.415599 88.604)
-		(end 197.415599 93.604)
-		(width 0.4)
-		(layer "B.Cu")
-		(net 5)
-	)
-	(segment
-		(start 92.049999 88.582)
-		(end 92.049999 93.582)
-		(width 0.4)
-		(layer "B.Cu")
-		(net 5)
-	)
-	(segment
-		(start 92.049999 93.582)
-		(end 98.279999 99.812)
-		(width 0.4)
-		(layer "B.Cu")
-		(net 5)
-	)
-	(segment
 		(start 141.315 92.575)
 		(end 141.315 91.66)
@@
 	)
 	(segment
-		(start 168.8 151.1)
-		(end 168.8 151.9)
+		(start 168.8 151.05)
+		(end 168.8 151.85)
 		(width 0.2)
 		(layer "F.Cu")
@@
 	)
 	(segment
-		(start 170.3 149.6)
-		(end 168.8 151.1)
+		(start 170.3 149.55)
+		(end 168.8 151.05)
 		(width 0.2)
 		(layer "F.Cu")
@@
 	)
 	(segment
-		(start 118.725 147.125)
-		(end 118.725 147.925)
+		(start 118.725 147.175)
+		(end 118.725 147.975)
 		(width 0.2)
 		(layer "F.Cu")
@@
 	)
 	(segment
-		(start 120.3 149.5)
-		(end 121.5 149.5)
+		(start 120.3 149.55)
+		(end 121.5 149.55)
 		(width 0.2)
 		(layer "F.Cu")
@@
 	)
 	(segment
-		(start 118.725 147.925)
-		(end 120.3 149.5)
+		(start 118.725 147.975)
+		(end 120.3 149.55)
 		(width 0.2)
 		(layer "F.Cu")
@@
 	)
 	(via
-		(at 121.5 149.5)
+		(at 121.5 149.55)
 		(size 0.6)
 		(drill 0.3)
@@
 	)
 	(segment
+		(start 121.5 149.55)
+		(end 121.55 149.55)
+		(width 0.2)
+		(layer "In1.Cu")
+		(net 12)
+	)
+	(segment
 		(start 156.7 149.8)
 		(end 179 127.5)
@@
 	)
 	(segment
-		(start 121.5 149.5)
+		(start 121.55 149.55)
 		(end 121.8 149.8)
 		(width 0.2)
@@
 	)
 	(segment
-		(start 97.938 114.7)
-		(end 86.3 103.062)
+		(start 156.1 114.7)
+		(end 98.7 114.7)
 		(width 0.2)
 		(layer "In1.Cu")
@@
 	)
 	(segment
-		(start 170.2 129.6)
-		(end 170.2 128.8)
+		(start 88.3316 104.3316)
+		(end 88.3316 103.084)
+		(width 0.2)
+		(layer "In1.Cu")
+		(net 51)
+	)
+	(segment
+		(start 98.7 114.7)
+		(end 88.3316 104.3316)
 		(width 0.2)
 		(layer "In1.Cu")
@@
 	)
 	(segment
-		(start 156.1 114.7)
-		(end 97.938 114.7)
+		(start 170.2 129.6)
+		(end 170.2 128.8)
 		(width 0.2)
 		(layer "In1.Cu")
@@
 	)
 	(segment
-		(start 153.951 102.451)
-		(end 103.418999 102.451)
+		(start 101.111699 96.5339)
+		(end 148.0339 96.5339)
 		(width 0.2)
 		(layer "In1.Cu")
@@
 	)
 	(segment
-		(start 176.2 124.7)
-		(end 153.951 102.451)
+		(start 100.311599 97.334)
+		(end 101.111699 96.5339)
 		(width 0.2)
 		(layer "In1.Cu")
@@
 	)
 	(segment
-		(start 103.418999 102.451)
-		(end 98.279999 97.312)
+		(start 148.0339 96.5339)
+		(end 176.2 124.7)
 		(width 0.2)
 		(layer "In1.Cu")
@@
 	)
 	(segment
-		(start 89.549999 88.582)
-		(end 89.549999 94.349999)
+		(start 105.049 107.049)
+		(end 91.581599 93.581599)
 		(width 0.2)
 		(layer "In1.Cu")
@@
 	)
 	(segment
-		(start 102.249 107.049)
-		(end 157.649 107.049)
+		(start 91.581599 93.581599)
+		(end 91.581599 88.604)
 		(width 0.2)
 		(layer "In1.Cu")
@@
 	)
 	(segment
-		(start 89.549999 94.349999)
-		(end 102.249 107.049)
+		(start 157.649 107.049)
+		(end 105.049 107.049)
 		(width 0.2)
 		(layer "In1.Cu")

Commit message: added tranceiver and joystick
Parts:
- removed AE1: Antenna, Connector_Coaxial:SMA_Amphenol_901-143_Horizontal
- removed REF** (x4): MountingHole_3.2mm_M3, MountingHole:MountingHole_3.2mm_M3
- added C23: 0.1uF, Capacitor_SMD:C_0402_1005Metric, F.Cu at (161.8, 129.5)
- added J4: Conn_Coaxial, Connector_Coaxial:SMA_Amphenol_901-143_Horizontal, F.Cu at (143.2, 69.1)
- added SW5: BTN_2, Connector_Wire:SolderWire-0.1sqmm_1x02_P3.6mm_D0.4mm_OD1mm, F.Cu at (160.1, 131.5)
- D1: footprint LED_THT:LED_D5.0mm -> LED_SMD:LED_0603_1608Metric
- J3: footprint Connector_JST:JST_PH_B4B-PH-K_1x04_P2.00mm_Vertical -> Connector_JST:JST_PH_S4B-PH-K_1x04_P2.00mm_Horizontal
- L4: footprint Inductor_SMD:L_7.3x7.3_H3.5 -> Inductor_SMD:L_6.3x6.3_H3
- SW4: value EStop -> BTN_1
- moved C26 3.03 mm to (161.8, 125.5)
- moved SW4 3.03 mm to (160.0, 127.5)
- moved C8 1.08 mm to (140.2, 85.4)
- moved C7 0.98 mm to (139.2, 85.4)
Connections:
- C26 pad 2: /ESTOP -> /BTN_1
- SW4 pad 2: /ESTOP -> /BTN_1
- U6 pad 18: /SX_BUSY -> /SX_RST
- U6 pad 19: /SX_DIO1 -> /SX_BUSY
- U6 pad 20: /SX_RST -> /SX_DIO1
- U6 pad 21: unconnected-(U6-IO17-Pad21) -> /BTN_1
- U6 pad 22: /ESTOP -> /BTN_2
Routing:
- net /BTN_1: track 0.00 -> 9.72 mm
- net /ESTOP: track 8.01 -> 0.00 mm
- net /BTN_2: track 0.00 -> 7.74 mm
- net /SX_RST: track 52.0 -> 49.5 mm, vias 2 -> 0
- net /SX_DIO1: track 49.2 -> 50.2 mm

Commit message: updated controller pcb
Parts:
- removed C1, C2: 0.1uF, Capacitor_SMD:C_0402_1005Metric
- removed C10: 39pF, Capacitor_SMD:C_0402_1005Metric
- removed C11, C12: 3.3pF, Capacitor_SMD:C_0402_1005Metric
- removed C3: 470nF, Capacitor_SMD:C_0402_1005Metric
- removed C7: 47nF, Capacitor_SMD:C_0402_1005Metric
- removed C8: 47pF, Capacitor_SMD:C_0402_1005Metric
- removed C9: 1nF, Capacitor_SMD:C_0402_1005Metric
- removed FL1: 0900FM15K0039, RF_Converter:Balun_Johanson_0900FM15K0039
- removed L1: 15uH, Inductor_SMD:L_0402_1005Metric
- removed L2: 47nH, Inductor_SMD:L_0402_1005Metric
- removed L3: 9.1nH, Inductor_SMD:L_0402_1005Metric
- removed R4: 100, Resistor_SMD:R_0402_1005Metric
- removed U2: SX1262IMLTRT, Package_DFN_QFN:QFN-24-1EP_4x4mm_P0.5mm_EP2.6x2.6mm
- removed U4: PE4259, Package_TO_SOT_SMD:SOT-363_SC-70-6
- removed Y2: 32MHz, Crystal:Crystal_SMD_3225-4Pin_3.2x2.5mm
- added J5: Tranceiver Boot/Rst, Connector_JST:JST_XH_B2B-XH-A_1x02_P2.50mm_Vertical, F.Cu at (133.3, 91.5)
- added REF**: MountingHole_2.7mm_M2.5, MountingHole:MountingHole_2.7mm_M2.5, F.Cu at (155.7, 67.5)
- added REF**: MountingHole_2.7mm_M2.5, MountingHole:MountingHole_2.7mm_M2.5, F.Cu at (130.7, 67.5)
- D1: footprint LED_SMD:LED_0603_1608Metric -> LED_THT:LED_D5.0mm
- J4: value Conn_Coaxial -> Tranceiver Data; footprint Connector_Coaxial:SMA_Amphenol_901-143_Horizontal -> Connector_JST:JST_XH_B4B-XH-A_1x04_P2.50mm_Vertical
- moved J4 22.7 mm to (146.8, 91.5), turned to 180 degrees
- moved TH1 7.00 mm to (143.2, 118.0)
- moved BT1 6.80 mm to (179.7, 106.0)
Connections:
- J4 pad 1: Net-(J4-In) -> +3.3V
- U6 pad 14: /SX_CS -> /STM32_RST
- U6 pad 15: /MOSI -> /STM32_BOOT
- U6 pad 16: /SCK -> unconnected-(U6-IO12-Pad16)
- U6 pad 17: /MISO -> unconnected-(U6-IO13-Pad17)
- U6 pad 18: /SX_RST -> unconnected-(U6-IO14-Pad18)
- U6 pad 19: /SX_BUSY -> unconnected-(U6-IO15-Pad19)
- U6 pad 20: /SX_DIO1 -> unconnected-(U6-IO16-Pad20)
- U6 pad 39: unconnected-(U6-TXD0-Pad39) -> /ESP_TX
- U6 pad 40: unconnected-(U6-RXD0-Pad40) -> /ESP_RX
Routing:
- net +3.3V: track 32.5 -> 321.1 mm, vias 10 -> 8
- net /ESP_TX: track 0.00 -> 68.1 mm, vias 0 -> 2
- net /ESP_RX: track 0.00 -> 67.6 mm, vias 0 -> 2
- net /STM32_BOOT: track 0.00 -> 55.8 mm, vias 0 -> 1
- net /STM32_RST: track 0.00 -> 55.5 mm, vias 0 -> 1
- net /BOOT: track 72.7 -> 127.2 mm, vias 2 -> 4
- net /SX_CS: track 50.6 -> 0.00 mm
- net /SX_DIO1: track 50.2 -> 0.00 mm
- net /SX_BUSY: track 49.7 -> 0.00 mm
- net /SCK: track 49.6 -> 0.00 mm, vias 2 -> 0
- net /SX_RST: track 49.5 -> 0.00 mm
- net /MISO: track 49.2 -> 0.00 mm
- net /MOSI: track 48.1 -> 0.00 mm
- net GND: track 69.3 -> 50.8 mm, vias 252 -> 177
- net /BAT_ADC: track 44.3 -> 56.0 mm
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- removed copper zone on In2.Cu, net +3.3V
- removed copper zone on In1.Cu, net GND
Other:
- copper layers 4 -> 2

Commit message: cleaning up controller pcb
Parts:
- J3: footprint Connector_JST:JST_PH_S4B-PH-K_1x04_P2.00mm_Horizontal -> Connector_JST:JST_XH_B4B-XH-A_1x04_P2.50mm_Vertical
Routing:
- net /BOOT: track 127.2 -> 112.7 mm, vias 4 -> 2
- net /JOY_2_BTN: track 100.8 -> 99.6 mm
- net /EN: track 22.0 -> 20.8 mm, vias 1 -> 0
- net /BAT_ADC: track 56.0 -> 55.0 mm
- net +3.3V: track 321.1 -> 320.6 mm, vias 8 -> 7

Commit message: updated cad
Parts:
- added REF**: MountingHole_3.2mm_M3, MountingHole:MountingHole_3.2mm_M3, F.Cu at (110.7, 149.6)
- added REF**: MountingHole_3.2mm_M3, MountingHole:MountingHole_3.2mm_M3, F.Cu at (110.7, 74.5)
- added REF**: SMA_Amphenol_901-144_Vertical, Connector_Coaxial:SMA_Amphenol_901-144_Vertical, F.Cu at (143.2, 69.5)
- added REF**: MountingHole_3.2mm_M3, MountingHole:MountingHole_3.2mm_M3, F.Cu at (175.7, 149.6)
- added REF**: MountingHole_3.2mm_M3, MountingHole:MountingHole_3.2mm_M3, F.Cu at (175.7, 74.5)
- moved REF** 0.50 mm to (155.2, 67.5)
- moved REF** 0.50 mm to (131.2, 67.5)
Routing:
- net GND: vias 177 -> 179
