File: hardware/transceiver/transceiver.kicad_pcb (KiCad board)
At the start: 4 copper layers, 30 x 30 mm, 50 parts, among them J1 Conn_01x04, J2 Conn_01x02, J3 Conn_Coaxial, J4 Conn_01x02, U1 SX1262IMLTRT, U2 AP2112K-3.3, U3 PE4259, U4 STM32U585CIUx, Y1 32MHz, Y2 Q13FC13500004, Y3 X322516MLB4SI

Commit message: added production files
Parts:
- BOOT: renamed from BOOT1; value Boot -> SW_Push
- L2: footprint Inductor_SMD:L_0402_1005Metric -> Inductor_SMD:L_0603_1608Metric
- R2, R3: value 1k -> 2K
- RESET: renamed from RESET1; value Reset -> SW_Push
- moved C7 2.24 mm to (130.2, 115.7), turned to 180 degrees
- moved L2 0.94 mm to (132.7, 115.6)
- renumbered C7 to C6, C6 to C7
Routing:
- net GND: track 66.8 -> 65.5 mm
- net Net-(U1-DCC_SW): track 2.38 -> 1.52 mm
Changed lines of the file:
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@@
 		(descr "Capacitor SMD 0603 (1608 Metric), square (rectangular) end terminal, IPC-7351 nominal, (Body size source: IPC-SM-782 page 76, https://www.pcb-3d.com/wordpress/wp-content/uploads/ipc-sm-782a_amendment_1_and_2.pdf), generated with kicad-footprint-generator")
 		(tags "capacitor")
-		(property "Reference" "C7"
+		(property "Reference" "C6"
 			(at 0 -1.43 0)
 			(layer "F.SilkS")
@@
 			)
 		)
-		(property "Value" "1k"
+		(property "Value" "2K"
 			(at 0 1.17 0)
 			(layer "F.Fab")
@@
 	(footprint "Capacitor_SMD:C_0402_1005Metric"
 		(layer "F.Cu")
-		(at 132.47 115.4)
+		(at 130.25 115.7 180)
 		(descr "Capacitor SMD 0402 (1005 Metric), square (rectangular) end terminal, IPC-7351 nominal, (Body size source: IPC-SM-782 page 76, https://www.pcb-3d.com/wordpress/wp-content/uploads/ipc-sm-782a_amendment_1_and_2.pdf), generated with kicad-footprint-generator")
 		(tags "capacitor")
-		(property "Reference" "C6"
+		(property "Reference" "C7"
 			(at 0 -1.16 0)
 			(layer "F.SilkS")
@@
 		(attr smd)
 		(fp_line
-			(start -0.107836 -0.36)
-			(end 0.107836 -0.36)
+			(start -0.107836 0.36)
+			(end 0.107836 0.36)
 			(stroke
 				(width 0.12)
@@
 		)
 		(fp_line
-			(start -0.107836 0.36)
-			(end 0.107836 0.36)
+			(start -0.107836 -0.36)
+			(end 0.107836 -0.36)
 			(stroke
 				(width 0.12)
@@
 		)
 		(fp_line
-			(start -0.91 -0.46)
-			(end 0.91 -0.46)
+			(start 0.91 0.46)
+			(end -0.91 0.46)
 			(stroke
 				(width 0.05)
@@
 		)
 		(fp_line
-			(start -0.91 0.46)
-			(end -0.91 -0.46)
+			(start 0.91 -0.46)
+			(end 0.91 0.46)
 			(stroke
 				(width 0.05)
@@
 		)
 		(fp_line
-			(start 0.91 -0.46)
-			(end 0.91 0.46)
+			(start -0.91 0.46)
+			(end -0.91 -0.46)
 			(stroke
 				(width 0.05)
@@
 		)
 		(fp_line
-			(start 0.91 0.46)
-			(end -0.91 0.46)
+			(start -0.91 -0.46)
+			(end 0.91 -0.46)
 			(stroke
 				(width 0.05)
@@
 		)
 		(fp_line
-			(start -0.5 -0.25)
-			(end 0.5 -0.25)
+			(start 0.5 0.25)
+			(end -0.5 0.25)
 			(stroke
 				(width 0.1)
@@
 		)
 		(fp_line
-			(start -0.5 0.25)
-			(end -0.5 -0.25)
+			(start 0.5 -0.25)
+			(end 0.5 0.25)
 			(stroke
 				(width 0.1)
@@
 		)
 		(fp_line
-			(start 0.5 -0.25)
-			(end 0.5 0.25)
+			(start -0.5 0.25)
+			(end -0.5 -0.25)
 			(stroke
 				(width 0.1)
@@
 		)
 		(fp_line
-			(start 0.5 0.25)
-			(end -0.5 0.25)
+			(start -0.5 -0.25)
+			(end 0.5 -0.25)
 			(stroke
 				(width 0.1)
@@
 		)
 		(pad "1" smd roundrect
-			(at -0.48 0)
+			(at -0.48 0 180)
 			(size 0.56 0.62)
 			(layers "F.Cu" "F.Mask" "F.Paste")
@@
 		)
 		(pad "2" smd roundrect
-			(at 0.48 0)
+			(at 0.48 0 180)
 			(size 0.56 0.62)
 			(layers "F.Cu" "F.Mask" "F.Paste")
@@
 			)
 		)
-		(property "Value" "1k"
+		(property "Value" "2K"
 			(at 0 1.17 0)
 			(layer "F.Fab")
@@
 		)
 	)
-	(footprint "Inductor_SMD:L_0402_1005Metric"
+	(footprint "Inductor_SMD:L_0603_1608Metric"
 		(layer "F.Cu")
-		(at 133.185 116.4 180)
-		(descr "Inductor SMD 0402 (1005 Metric), square (rectangular) end terminal, IPC-7351 nominal, (Body size source: http://www.tortai-tech.com/upload/download/2011102023233369053.pdf), generated with kicad-footprint-generator")
+		(at 132.7 115.6 180)
+		(descr "Inductor SMD 0603 (1608 Metric), square (rectangular) end terminal, IPC-7351 nominal, (Body size source: http://www.tortai-tech.com/upload/download/2011102023233369053.pdf), generated with kicad-footprint-generator")
 		(tags "inductor")
 		(property "Reference" "L2"
-			(at 0 -1.17 0)
+			(at 0 -1.43 180)
 			(layer "F.SilkS")
 			(hide yes)
@@
 		)
 		(property "Value" "15uH"
-			(at 0 1.17 0)
+			(at 0 1.43 180)
 			(layer "F.Fab")
 			(effects
@@
 		)
 		(property "Datasheet" "~"
-			(at 0 0 0)
+			(at 0 0 180)
 			(layer "F.Fab")
 			(hide yes)
@@
 		)
 		(property "Description" "Inductor"
-			(at 0 0 0)
+			(at 0 0 180)
 			(layer "F.Fab")
 			(hide yes)
@@
 		(attr smd)
 		(fp_line
-			(start 0.93 0.47)
-			(end -0.93 0.47)
+			(start -0.162779 0.51)
+			(end 0.162779 0.51)
+			(stroke
+				(width 0.12)
+				(type solid)
+			)
+			(layer "F.SilkS")
+		)
+		(fp_line
+			(start -0.162779 -0.51)
+			(end 0.162779 -0.51)
+			(stroke
+				(width 0.12)
+				(type solid)
+			)
+			(layer "F.SilkS")
+		)
+		(fp_line
+			(start 1.48 0.73)
+			(end -1.48 0.73)
 			(stroke
 				(width 0.05)
@@
 		)
 		(fp_line
-			(start 0.93 -0.47)
-			(end 0.93 0.47)
+			(start 1.48 -0.73)
+			(end 1.48 0.73)
 			(stroke
 				(width 0.05)
@@
 		)
 		(fp_line
-			(start -0.93 0.47)
-			(end -0.93 -0.47)
+			(start -1.48 0.73)
+			(end -1.48 -0.73)
 			(stroke
 				(width 0.05)
@@
 		)
 		(fp_line
-			(start -0.93 -0.47)
-			(end 0.93 -0.47)
+			(start -1.48 -0.73)
+			(end 1.48 -0.73)
 			(stroke
 				(width 0.05)
@@
 		)
 		(fp_line
-			(start 0.5 0.25)
-			(end -0.5 0.25)
+			(start 0.8 0.4)
+			(end -0.8 0.4)
 			(stroke
 				(width 0.1)
@@
 		)
 		(fp_line
-			(start 0.5 -0.25)
-			(end 0.5 0.25)
+			(start 0.8 -0.4)
+			(end 0.8 0.4)
 			(stroke
 				(width 0.1)
@@
 		)
 		(fp_line
-			(start -0.5 0.25)
-			(end -0.5 -0.25)
+			(start -0.8 0.4)
+			(end -0.8 -0.4)
 			(stroke
 				(width 0.1)
@@
 		)
 		(fp_line
-			(start -0.5 -0.25)
-			(end 0.5 -0.25)
+			(start -0.8 -0.4)
+			(end 0.8 -0.4)
 			(stroke
 				(width 0.1)
@@
 		)
 		(fp_text user "${REFERENCE}"
-			(at 0 0 0)
+			(at 0 0 180)
 			(layer "F.Fab")
 			(effects
 				(font
-					(size 0.25 0.25)
-					(thickness 0.04)
+					(size 0.4 0.4)
+					(thickness 0.06)
 				)
 			)
 		)
 		(pad "1" smd roundrect
-			(at -0.485 0 180)
-			(size 0.59 0.64)
+			(at -0.7875 0 180)
+			(size 0.875 0.95)
 			(layers "F.Cu" "F.Mask" "F.Paste")
 			(roundrect_rratio 0.25)
@@
 		)
 		(pad "2" smd roundrect
-			(at 0.485 0 180)
-			(size 0.59 0.64)
+			(at 0.7875 0 180)
+			(size 0.875 0.95)
 			(layers "F.Cu" "F.Mask" "F.Paste")
 			(roundrect_rratio 0.25)
@@
 		)
 		(embedded_fonts no)
-		(model "${KICAD9_3DMODEL_DIR}/Inductor_SMD.3dshapes/L_0402_1005Metric.step"
+		(model "${KICAD9_3DMODEL_DIR}/Inductor_SMD.3dshapes/L_0603_1608Metric.step"
 			(offset
 				(xyz 0 0 0)
@@
 		(descr "http://www.alps.com/prod/info/E/HTML/Tact/SurfaceMount/SKRK/SKRKAHE020.html")
 		(tags "SMD SMT button")
-		(property "Reference" "RESET1"
+		(property "Reference" "RESET"
 			(at 3.4 -0.7 180)
 			(layer "F.SilkS")
@@
 			)
 		)
-		(property "Value" "Reset"
+		(property "Value" "SW_Push"
 			(at 0 2.5 90)
 			(layer "F.Fab")
@@
 		(descr "http://www.alps.com/prod/info/E/HTML/Tact/SurfaceMount/SKRK/SKRKAHE020.html")
 		(tags "SMD SMT button")
-		(property "Reference" "BOOT1"
+		(property "Reference" "BOOT"
 			(at 3.5 0.4 180)
 			(layer "F.SilkS")
@@
 			)
 		)
-		(property "Value" "Boot"
+		(property "Value" "SW_Push"
 			(at 0 2.5 90)
 			(layer "F.Fab")
@@
 	)
 	(segment
-		(start 132.95 115.4)
-		(end 132.95 114.15)
-		(width 0.2)
-		(layer "F.Cu")
-		(net 1)
-	)
-	(segment
 		(start 145.089949 104.2075)
 		(end 144.369949 104.2075)
@@
 	)
 	(segment
-		(start 132.95 114.15)
-		(end 133.0125 114.0875)
-		(width 0.2)
-		(layer "F.Cu")
-		(net 1)
-	)
-	(segment
 		(start 143.589949 104.9875)
 		(end 143.589949 103.910051)
@@
 	)
 	(via
-		(at 130 117.5)
+		(at 129.5 116.5)
 		(size 0.6)
 		(drill 0.3)
@@
 	)
 	(via
-		(at 131.5125 116.9)
+		(at 132.2 116.8)
 		(size 0.6)
 		(drill 0.3)
@@
 	)
 	(via
-		(at 129.0125 115.9)
+		(at 128.9 115.9)
 		(size 0.6)
 		(drill 0.3)
@@
 	)
 	(via
-		(at 132.2625 117.4)
+		(at 133 116.8)
 		(size 0.6)
 		(drill 0.3)
@@
 	)
 	(via
-		(at 130.7625 116.15)
+		(at 130.3 116.7)
 		(size 0.6)
 		(drill 0.3)
@@
 	)
 	(via
-		(at 133.2625 117.65)
+		(at 133.8 117.1)
 		(size 0.6)
 		(drill 0.3)
@@
 	)
 	(via
-		(at 128.5 118.75)
+		(at 129.8 118.2)
 		(size 0.6)
 		(drill 0.3)
@@
 	)
 	(via
-		(at 130.0125 115.9)
+		(at 131.2 116.8)
 		(size 0.6)
 		(drill 0.3)
@@
 	)
 	(segment
-		(start 131.99 115.69)
-		(end 132.7 116.4)
+		(start 131.9125 115.6)
+		(end 130.83 115.6)
 		(width 0.2)
 		(layer "F.Cu")
@@
 	)
 	(segment
-		(start 131.99 114.61)
-		(end 132.5125 114.0875)
+		(start 130.83 115.6)
+		(end 130.73 115.7)
 		(width 0.2)
 		(layer "F.Cu")
@@
 	)
 	(segment
-		(start 131.99 115.4)
-		(end 131.99 114.61)
+		(start 132.5125 114.0875)
+		(end 132.5125 115)
 		(width 0.2)
 		(layer "F.Cu")
@@
 	)
 	(segment
-		(start 131.99 115.4)
-		(end 131.99 115.69)
+		(start 132.5125 115)
+		(end 131.9125 115.6)
 		(width 0.2)
 		(layer "F.Cu")
@@
 	)
 	(segment
-		(start 133.5125 114.499999)
-		(end 133.6125 114.599999)
-		(width 0.2)
-		(layer "F.Cu")
-		(net 16)
-	)
-	(segment
-		(start 133.6125 116.3425)
-		(end 133.67 116.4)
-		(width 0.2)
-		(layer "F.Cu")
-		(net 16)
-	)
-	(segment
-		(start 133.6125 114.599999)
-		(end 133.6125 116.3425)
+		(start 133.5125 115.575)
+		(end 133.4875 115.6)
 		(width 0.2)
 		(layer "F.Cu")
@@
 	(segment
 		(start 133.5125 114.0875)
-		(end 133.5125 114.499999)
+		(end 133.5125 115.575)
 		(width 0.2)
 		(layer "F.Cu")

Commit message: added version to silkscreen
Other:
- board text added: "Transceiver V1.0"
Changed lines of the file:
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@@
 		(layer "Edge.Cuts")
+	)
+	(gr_text "Transceiver V1.0"
+		(at 154.5 100.5 90)
+		(layer "B.SilkS")
+		(effects
+			(font
+				(size 1 1)
+				(thickness 0.2)
+				(bold yes)
+			)
+			(justify left bottom mirror)
+		)
 	)
 	(segment
